File: kicad_files/37NJU22_emul_RPPICO_card.kicad_pcb (KiCad board)
At the start: 2 copper layers, 54 x 85.7 mm, 60 parts, among them CN1 HDMI, J1 VGA, J10 Conn_01x02, J11 Conn_01x01, J12 Audio OUT, J13 Audio IN, J2 EXT, J3 Micro_SD_Card, J4 Conn_SD, J5 PWR, J6 UART, J7 Mini-DIN-6, J8 IN_A, J9 IN_A, Q3 BC850, Q4 BC850, U1 raspberrypi-pico-module

Commit message: .
Other:
- board text added: "32NJU23"
- board text removed: "37NJU23"
Changed lines of the file:
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@@
       (layerselection 0x00010fc_ffffffff)
       (disableapertmacros false)
-      (usegerberextensions false)
-      (usegerberattributes true)
-      (usegerberadvancedattributes true)
-      (creategerberjobfile true)
+      (usegerberextensions true)
+      (usegerberattributes false)
+      (usegerberadvancedattributes false)
+      (creategerberjobfile false)
       (svguseinch false)
       (svgprecision 6)
@@
       (psa4output false)
       (plotreference true)
-      (plotvalue true)
+      (plotvalue false)
       (plotinvisibletext false)
       (sketchpadsonfab false)
-      (subtractmaskfromsilk false)
+      (subtractmaskfromsilk true)
       (outputformat 1)
       (mirror false)
       (drillshape 0)
       (scaleselection 1)
-      (outputdirectory "GERBER_OUT/")
+      (outputdirectory "gerber/")
     )
   )
@@
     (fp_line (start -1.67 39.16) (end -1.67 39.58) (layer "F.SilkS") (width 0.12))
     (fp_line (start 19.45 1.06) (end 19.45 1.48) (layer "F.SilkS") (width 0.12))
-    (fp_arc (start 19.42 49.32) (mid 19.213497 49.588778) (end 18.89 49.69) (layer "F.SilkS") (width 0.12))
-    (fp_arc (start 18.89 -1.43) (mid 19.213484 -1.328785) (end 19.42 -1.06) (layer "F.SilkS") (width 0.12))
+    (fp_arc (start 19.42 49.32) (mid 19.213487 49.588772) (end 18.89 49.69) (layer "F.SilkS") (width 0.12))
+    (fp_arc (start 18.89 -1.43) (mid 19.213502 -1.328793) (end 19.42 -1.06) (layer "F.SilkS") (width 0.12))
     (fp_arc (start -1.11 49.69) (mid -1.433508 49.588809) (end -1.64 49.32) (layer "F.SilkS") (width 0.12))
     (fp_arc (start -1.64 -1.06) (mid -1.433508 -1.328808) (end -1.11 -1.43) (layer "F.SilkS") (width 0.12))
@@
     (effects (font (size 1 1) (thickness 0.15)) (justify mirror))
   )
-  (gr_text "37NJU23" (at 56.55 112.25) (layer "B.SilkS")
+  (gr_text "32NJU23" (at 56.55 112.25) (layer "B.SilkS")
     (effects (font (size 1 1) (thickness 0.15)) (justify mirror))
   )
